File: Hardware/Satellite_Transceiver_Breakout__Swarm_M138.sch (EAGLE design)
At the start: 61 parts, among them Q2 20V/4.2A/52mΩ/1.4W, Q4 20V/4.2A/52mΩ/1.4W, U1 CH340E_MSOP10, U2 SWARM_M138_TRANSCEIVER_MAIN, U3 3.3V

Commit message: Adds more measures, adds shield jumper, reduces polygon isolate to .007
* Adds new net class for RF traces between u.FL and SMA connectors to keep .01 isolate on those
particular traces
* Removes Sparkx silk and adds SparkFun silk
* Adds "Revised by" text
* Center aligns all schematic text
Parts:
- removed LOGO3: OSHW-LOGOM, SparkFun-Aesthetics:OSHW-LOGOM
- removed U$1, U$2: SPARKX-LOGO5, SparkX:SPARKX-LOGO5
- added LOGO4: SFE_LOGO_NAME_FLAME.1_INCH, SparkFun-Aesthetics:SFE_LOGO_NAME_FLAME.1_INCH
- added SHLD: JUMPER-SMT_2_NC_TRACE_SILK, SparkFun-Jumpers:JUMPER-SMT_2_NC_TRACE_SILK
Connections:
- new net SHLD: J1.SHLD, SHLD.2
- net GND: now also SHLD.1; no longer J1.SHLD
- net N$13: now also Q1G2.C; no longer Q1G$2.C
- net N$15: now also Q3G1.B, Q3G1.C, Q3G2.B; no longer Q3G$1.B, Q3G$1.C, Q3G$2.B
- net N$28: now also Q3G2.C; no longer Q3G$2.C
- net N$5: now also Q1G1.B, Q1G1.C, Q1G2.B; no longer Q1G$1.B, Q1G$1.C, Q1G$2.B
- net VCC: now also Q1G2.E, Q3G2.E; no longer Q1G$2.E, Q3G$2.E
- net VIN: now also Q3G1.E; no longer Q3G$1.E
- net V_USB_2: now also Q1G1.E; no longer Q1G$1.E
Other:
- note added: "Cut "SHLD" to disconnect shield from ground."
- note added: "Cut Jumpers to isolate UART lines from CH340C"
- note added: "Revised By: Elias Santistevan"
- note added: "Sattelite Transceiver - Swarm M138"
- note added: "v10"
- note removed: "Swarm M138"
- note removed: "x03"
- moved on the sheet: BYP, D1, F1, J1, J2, JP1, R1, R2, RXI, TXO
